File: EXTENSION_BOARD/EXTENSION_BOARD.kicad_pcb (KiCad board)
At the start: 2 copper layers, 25 parts, among them IC1 Baro, IC2 ICM-20608-G, J1 EXTOUT, J2 PWM, U1 Teensy4.0, U2 COM-15809

Commit message: Update EXTENSION_BOARD.kicad_pcb
Parts:
- added REF**: MountingHole_3.2mm_M3, MountingHole:MountingHole_3.2mm_M3, F.Cu at (93.5, 106.3)
- added REF**: MountingHole_3.2mm_M3, MountingHole:MountingHole_3.2mm_M3, F.Cu at (136.4, 106.3)
- added REF**: MountingHole_3.2mm_M3, MountingHole:MountingHole_3.2mm_M3, F.Cu at (136.5, 83.6)
- C1, C4, C6, R1, R7: moved to B.Cu
- D1, D2, D3, D4, D5: footprint digikey-footprints:LED_2-SMD_No_Lead_1.7x0.8mm -> KRTEK_V2:LED_2-SMD_No_Lead_1.7x0.8mm
- IC1: footprint SamacSys_Parts:MS561101BA03-50 -> KRTEK_V2:MS561101BA03-50
- IC2: footprint SamacSys_Parts:PULL-BACK-QFN-16 -> KRTEK_V2:PULL-BACK-QFN-16
- J1: footprint SamacSys_Parts:2828345 -> KRTEK_V2:2828345
- J2: footprint SamacSys_Parts:282834-2_1 -> KRTEK_V2:282834-2_1
- LS1: footprint SamacSys_Parts:PS1240P02BT -> KRTEK_V2:CST931AP
- U1: footprint teensy:Teensy40 -> EXTENSION:Teensy40
- U2: footprint digikey-footprints:SOIC-8_W5.6mm -> KRTEK_V2:SOIC-8_W5.6mm
- moved C2 40.3 mm to (85.2, 67.0)
- moved C3 40.3 mm to (85.1, 64.5)
- moved C5 40.3 mm to (81.7, 72.0)
- moved IC2 40.3 mm to (85.3, 70.6)
- moved C6 38.8 mm to (114.7, 103.3), turned to 90 degrees
- moved R7 38.7 mm to (117.7, 103.3), turned to 90 degrees
- moved U2 35.0 mm to (116.0, 103.4), turned to 180 degrees
- moved J1 27.4 mm to (136.6, 89.9), turned to 270 degrees
- moved J2 16.5 mm to (130.6, 83.4), turned to 180 degrees
- moved C1 13.5 mm to (128.6, 94.4), turned to 270 degrees
- moved C4 13.1 mm to (131.0, 94.5), turned to 90 degrees
- moved LS1 12.1 mm to (123.7, 103.6), turned to 270 degrees
- moved D2 11.8 mm to (100.3, 100.4)
- moved R4 11.8 mm to (103.9, 101.8)
- moved R6 11.8 mm to (111.3, 101.9)
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