File: EXTENSION_BOARD/EXTENSION_BOARD.kicad_pcb (KiCad board)
At the start: 2 copper layers, 50 x 32 mm, 39 parts, among them IC1 TeensyBuffer - 74AHCV541ABQX, IC2 Baro - MS561101BA03-50, J1 EXTIN, J2 BATT, J3 PWM, J5 EXTOUT, U1 Flash - COM-15809, U2 Teensy4.0, U3 MJD148J

Commit message: duh
Routing:
- net GND: vias 9 -> 10
Changed lines of the file:
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@@
   (general
     (thickness 1.6)
-    (drawings 11)
-    (tracks 370)
+    (drawings 13)
+    (tracks 371)
     (zones 0)
     (modules 39)
@@
     )
   )
+  (dimension 49.9872 (width 0.15) (layer Dwgs.User)
+    (gr_text "49.987 mm" (at 115.004009 118.430397 0.002911370908) (layer Dwgs.User)
+      (effects (font (size 1 1) (thickness 0.15)))
+    )
+    (feature1 (pts (xy 139.99718 109.98962) (xy 139.997573 117.715548)))
+    (feature2 (pts (xy 90.00998 109.99216) (xy 90.010373 117.718088)))
+    (crossbar (pts (xy 90.010343 117.131667) (xy 139.997543 117.129127)))
+    (arrow1a (pts (xy 139.997543 117.129127) (xy 138.871069 117.715605)))
+    (arrow1b (pts (xy 139.997543 117.129127) (xy 138.871009 116.542764)))
+    (arrow2a (pts (xy 90.010343 117.131667) (xy 91.136877 117.71803)))
+    (arrow2b (pts (xy 90.010343 117.131667) (xy 91.136817 116.545189)))
+  )
+  (dimension 31.98876 (width 0.15) (layer Dwgs.User)
+    (gr_text "31.989 mm" (at 150.301052 93.993604 -89.9909011) (layer Dwgs.User)
+      (effects (font (size 1 1) (thickness 0.15)))
+    )
+    (feature1 (pts (xy 139.99464 78.00086) (xy 149.584933 77.999337)))
+    (feature2 (pts (xy 139.99972 109.98962) (xy 149.590013 109.988097)))
+    (crossbar (pts (xy 149.003592 109.98819) (xy 148.998512 77.99943)))
+    (arrow1a (pts (xy 148.998512 77.99943) (xy 149.585112 79.125841)))
+    (arrow1b (pts (xy 148.998512 77.99943) (xy 148.41227 79.126027)))
+    (arrow2a (pts (xy 149.003592 109.98819) (xy 149.589834 108.861593)))
+    (arrow2b (pts (xy 149.003592 109.98819) (xy 148.416992 108.861779)))
+  )
   (gr_line (start 90 78) (end 90 110) (layer Edge.Cuts) (width 0.15))
   (gr_line (start 90 110) (end 140 110) (layer Edge.Cuts) (width 0.15))
@@
   (via (at 127.55372 95.91548) (size 0.8) (drill 0.4) (layers F.Cu B.Cu) (net 1))
   (via (at 128.0033 91.4908) (size 0.8) (drill 0.4) (layers F.Cu B.Cu) (net 1))
+  (via (at 91.78798 103.9114) (size 0.8) (drill 0.4) (layers F.Cu B.Cu) (net 1))
   (via (at 101.64572 102.98176) (size 0.8) (drill 0.4) (layers F.Cu B.Cu) (net 2))
   (segment (start 101.6381 102.97414) (end 101.64572 102.98176) (width 0.25) (layer F.Cu) (net 2))

Commit message: last commit
Other:
- net class Default removed
