File: EXTENSION_BOARD/EXTENSION_BOARD.sch (KiCad schematic (older format))
At the start: 25 parts, among them IC1 Baro, IC2 ICM-20608-G, J1 EXTOUT, J2 PWM, U1 Teensy4.0, U2 COM-15809

Commit message: Update EXTENSION_BOARD.sch
Parts:
- LS1: footprint KRTEK_V2:PS1240P02BT -> KRTEK_V2:CST931AP
Changed lines of the file:
@@
 F 0 "LS1" H 9478 1296 50  0000 L CNN
 F 1 "Buzzer" H 9478 1205 50  0000 L CNN
-F 2 "KRTEK_V2:PS1240P02BT" H 9500 1400 50  0001 L CNN
+F 2 "KRTEK_V2:CST931AP" H 9500 1400 50  0001 L CNN
 F 3 "https://product.tdk.com/system/files/dam/doc/product/sw_piezo/sw_piezo/piezo-buzzer/catalog/piezoelectronic_buzzer_ps_en.pdf" H 9500 1300 50  0001 L CNN
 F 4 "Piezoelectric Buzzers, Sound Pressure Level=60dB min, Freq.=4000Hz nom" H 9500 1200 50  0001 L CNN "Description"
