File: EXTENSION_BOARD/EXTENSION_BOARD.sch (KiCad schematic (older format))
At the start: 25 parts, among them IC1 Baro, IC2 ICM-20608-G, J1 EXTOUT, J2 PWM, U1 Teensy4.0, U2 COM-15809

Commit message: worked
Parts:
- removed J1: EXTOUT, KRTEK_V2:2828345, symbol SamacSys_Parts:282834-5
- removed J2: PWM, KRTEK_V2:282834-2_1, symbol SamacSys_Parts:282834-2
- added C7, C8, C9: 0.1uF, Capacitor_SMD:C_0603_1608Metric, symbol Device:C
- added IC3: MAX22700EASA+, EXTENSION:SOIC127P600X175-8N, symbol EXTENSION:MAX22700EASA+
- added IC4: TeensyBuffer, EXTENSION:QFN50P250X450X100-21N-D, symbol EXTENSION:74AHCV541ABQX
- added J1: BATT, EXTENSION:5055670281, symbol EXTENSION:505567-0281
- added J2: 505567-0671, EXTENSION:5055670671, symbol EXTENSION:505567-0671
- added J3: PWM, EXTENSION:5055670281, symbol EXTENSION:505567-0281
- added J4: EXTOUT, EXTENSION:5055670571, symbol EXTENSION:505567-0571
- added U3: MOSBuzzer, EXTENSION:TSOT-23, symbol EXTENSION:BSH105,235
- U1: footprint EXTENSION:Teensy40 -> EXTENSION:Teensy40_EXT
Connections:
- net labels added: HMISO, HMOSI, HSCK, MOSBuzzer, TBUZZ1, TBUZZ2, TBuzzer, TGLED1, TGLED2, TYLED1, TYLED2, VIN
- net labels removed: GTLED2
- wire segments 97 -> 144
Other:
- moved on the sheet: C6, R7, U2
