File: EXTENSION_BOARD/EXTENSION_BOARD.sch (KiCad schematic (older format))
At the start: 33 parts, among them IC1 Baro, IC2 ICM-20608-G, IC3 MAX22700EASA+, IC4 TeensyBuffer, J1 BATT, J2 505567-0671, J3 PWM, J4 EXTOUT, U1 Teensy4.0, U2 COM-15809, U3 MOSBuzzer

Commit message: Worked again
Parts:
- removed C2, C8, C9: 0.1uF, Capacitor_SMD:C_0603_1608Metric, symbol Device:C
- removed C5: 0.47uF, Capacitor_SMD:C_0603_1608Metric, symbol Device:C
- removed IC2: ICM-20608-G, KRTEK_V2:PULL-BACK-QFN-16, symbol SamacSys_Parts:ICM-20608-G
- removed IC3: MAX22700EASA+, EXTENSION:SOIC127P600X175-8N, symbol EXTENSION:MAX22700EASA+
- added AC1: Accel - H3LIS331DLTR, EXTENSION:LIS3DHTR, symbol EXTENSION:H3LIS331DLTR
- added D6, D7, D8, D9: DIODE, Diode_SMD:D_0603_1608Metric, symbol Simulation_SPICE:DIODE
- added R2, R3, R6: 10k, Resistor_SMD:R_0603_1608Metric, symbol Device:R
- added R5: 500, Resistor_SMD:R_0603_1608Metric, symbol Device:R
- C2: renamed from C1; value 100nF -> 0.1uF
- C3: value 10nF -> 0.1uF
- C4: value 2.2uF -> 10uF
- IC1: renamed from IC4; value TeensyBuffer -> TeensyBuffer - 74AHCV541ABQX
- IC2: renamed from IC1; value Baro -> Baro - MS561101BA03-50
- J1: renamed from J2; value 505567-0671 -> EXTIN
- LS1: value Buzzer -> Buzzer - CST-931AP
- R7: renamed from R2; value 740 -> 500
- U1: renamed from U2; value COM-15809 -> Flash - COM-15809
- U3: value MOSBuzzer -> MOSBuzzer - BSH105,235
- renumbered C6 to C1, C7 to C5, J1 to J2, R7 to R1, R5 to R10, R6 to R11, R1 to R4, R3 to R8, R4 to R9, U1 to U2
Connections:
- net labels added: +3.3V, Accel_INT1, Accel_INT2, Accel_SCL, Accel_SDA, Baro_SCLK, Baro_SDA, HFREE, HRX, HTX, INFREE1, INFREE2, OPYRO1, OPYRO2, OUTFREE1, OUTFREE2, TPyro1OUT, TPyro2OUT
- net labels removed: 3V3, CS_Baro, CS_IMU, FSYNC, HMISO, HMOSI, HSCK, INT, MOSBuzzer, RESV, SDI, SDO, VCC
- wire segments 144 -> 159
- no-connect marks 0 -> 2
Other:
- moved on the sheet: C1, C2, C5, D1, D2, D3, D4, D5, IC1, IC2, LS1, R1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

Commit message: Sent schematics to review
Parts:
- removed R6: 10k, Resistor_SMD:R_0603_1608Metric, symbol Device:R
- removed U3: MOSBuzzer - BSH105,235, EXTENSION:TSOT-23, symbol EXTENSION:BSH105,235
- added U3: MJD148J, Package_TO_SOT_SMD:TO-252-2, symbol EXTENSION:MJD148J
- R5: value 500 -> 10k
Connections:
- net +3V3: now also LS1.1, R4.1
- net Buzzer: now also LS1.2, R4.2, U3.2 (mb); no longer LS1.1, R4.1
- net GND: now also U3.3 (Emitter); no longer LS1.2, R4.2
- net HFREE: now also U2.30 (23_A9_CRX1_MCLK1)
- net at R5.1: now also U3.1 (Base)
Other:
- note added: "Accelerometer\nCommunicate I2C\n"
- note added: "Baro\ncommunicate I2C"
- note added: "Both Iacoboard and Teensy can fire pyros\nDiodes just to prevent them firing in each other"
- note added: "Buffer to use LEDs + optocoupler with Teensy"
- note added: "Buzzer + BJT"
- note added: "LEDs debug"
- note added: "Les connecteurs Mikro Lock"
- note added: "The one used by BPS space.\nNever used flash so hopefully it works :p\n"
- moved on the sheet: AC1, C3, C4, C5, D1, D2, D3, D4, D5, D6, D7, D8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

Commit message: t
Parts:
- removed J4: EXTOUT, EXTENSION:5055670571, symbol EXTENSION:505567-0571
- added J5: EXTOUT, EXTENSION:5055670671, symbol EXTENSION:505567-0671
Connections:
- net +3V3: now also J5.1
- net GND: now also J5.2
- net OPYRO1: now also J5.5
- net OPYRO2: now also J5.6
- net BUZZ1 renamed OUTFREE4
- net BUZZ2 renamed OUTFREE3
- net TBUZZ1 renamed INFREE4
- net INFREE4: no longer U2.8 (6_OUT1D)
- net TBUZZ2 renamed INFREE3
- net INFREE3: no longer U2.9 (7_RX2_OUT1A)
- new net PDECT1: J5.3, U2.8 (6_OUT1D)
- new net PDECT2: J5.4, U2.9 (7_RX2_OUT1A)
Other:
- moved on the sheet: J2
Changed lines of the file:
@@
 	3500 3450 3300 3450
-$Comp
-L EXTENSION:505567-0571 J4
-U 1 1 618D57EA
-P 10200 5100
-F 0 "J4" H 10600 5365 50  0000 C CNN
-F 1 "EXTOUT" H 10600 5274 50  0000 C CNN
-F 2 "EXTENSION:5055670571" H 10850 5200 50  0001 L CNN
-F 3 "https://www.molex.com/pdm_docs/sd/5055670571_sd.pdf" H 10850 5100 50  0001 L CNN
-F 4 "Molex Micro-Lock PLUS 505567, 1.25mm Pitch, 5 Way, 1 Row, Right Angle PCB Header, Surface Mount" H 10850 5000 50  0001 L CNN "Description"
-F 5 "3" H 10850 4900 50  0001 L CNN "Height"
-F 6 "538-505567-0571" H 10850 4800 50  0001 L CNN "Mouser Part Number"
-F 7 "https://www.mouser.co.uk/ProductDetail/Molex/505567-0571?qs=gt1LBUVyoHnJxHrzoS78pw%3D%3D" H 10850 4700 50  0001 L CNN "Mouser Price/Stock"
-F 8 "Molex" H 10850 4600 50  0001 L CNN "Manufacturer_Name"
-F 9 "505567-0571" H 10850 4500 50  0001 L CNN "Manufacturer_Part_Number"
-	1    10200 5100
-	1    0    0    -1
-$EndComp
 $Comp
 L EXTENSION:505567-0281 J3
@@
 	10050 6300 10100 6300
 $Comp
-L power:GND #PWR034
-U 1 1 618E3668
-P 10200 5050
-F 0 "#PWR034" H 10200 4800 50  0001 C CNN
-F 1 "GND" V 10205 4922 50  0000 R CNN
-F 2 "" H 10200 5050 50  0001 C CNN
-F 3 "" H 10200 5050 50  0001 C CNN
-	1    10200 5050
-	-1   0    0    1
-$EndComp
-Wire Wire Line
-	10150 5500 10200 5500
-Text GLabel 10150 5300 0    50   Input ~ 0
-BUZZ2
-Wire Wire Line
-	10150 5400 10200 5400
-Text GLabel 10150 5200 0    50   Input ~ 0
-BUZZ1
-Text GLabel 10150 5500 0    50   Input ~ 0
-OPYRO2
-Text GLabel 10150 5400 0    50   Input ~ 0
-OPYRO1
-Wire Wire Line
-	10150 5200 10200 5200
-Wire Wire Line
-	10150 5300 10200 5300
-$Comp
 L EXTENSION:505567-0281 J2
 U 1 1 61906994
-P 9950 4500
-F 0 "J2" H 10400 4765 50  0000 C CNN
-F 1 "BATT" H 10400 4674 50  0000 C CNN
-F 2 "EXTENSION:5055670281" H 10700 4600 50  0001 L CNN
-F 3 "https://www.molex.com/pdm_docs/sd/5055670281_sd.pdf" H 10700 4500 50  0001 L CNN
-F 4 "Headers & Wire Housings MicroLockPlus 1.25MM RA HDR SR 2P BLK GLD" H 10700 4400 50  0001 L CNN "Description"
-F 5 "3.9" H 10700 4300 50  0001 L CNN "Height"
-F 6 "538-505567-0281" H 10700 4200 50  0001 L CNN "Mouser Part Number"
-F 7 "https://www.mouser.co.uk/ProductDetail/Molex/505567-0281?qs=gt1LBUVyoHmc7tfcrPDm5A%3D%3D" H 10700 4100 50  0001 L CNN "Mouser Price/Stock"
-F 8 "Molex" H 10700 4000 50  0001 L CNN "Manufacturer_Name"
-F 9 "505567-0281" H 10700 3900 50  0001 L CNN "Manufacturer_Part_Number"
-	1    9950 4500
-	1    0    0    -1
-$EndComp
-Text GLabel 9750 4600 0    50   Input ~ 0
+P 10000 4200
+F 0 "J2" H 10450 4465 50  0000 C CNN
+F 1 "BATT" H 10450 4374 50  0000 C CNN
+F 2 "EXTENSION:5055670281" H 10750 4300 50  0001 L CNN
+F 3 "https://www.molex.com/pdm_docs/sd/5055670281_sd.pdf" H 10750 4200 50  0001 L CNN
+F 4 "Headers & Wire Housings MicroLockPlus 1.25MM RA HDR SR 2P BLK GLD" H 10750 4100 50  0001 L CNN "Description"
+F 5 "3.9" H 10750 4000 50  0001 L CNN "Height"
+F 6 "538-505567-0281" H 10750 3900 50  0001 L CNN "Mouser Part Number"
+F 7 "https://www.mouser.co.uk/ProductDetail/Molex/505567-0281?qs=gt1LBUVyoHmc7tfcrPDm5A%3D%3D" H 10750 3800 50  0001 L CNN "Mouser Price/Stock"
+F 8 "Molex" H 10750 3700 50  0001 L CNN "Manufacturer_Name"
+F 9 "505567-0281" H 10750 3600 50  0001 L CNN "Manufacturer_Part_Number"
+	1    10000 4200
+	1    0    0    -1
+$EndComp
+Text GLabel 9800 4300 0    50   Input ~ 0
 VIN
 Wire Wire Line
-	9900 4500 9950 4500
+	9950 4200 10000 4200
 $Comp
 L power:GND #PWR033
 U 1 1 6190D110
-P 9900 4500
-F 0 "#PWR033" H 9900 4250 50  0001 C CNN
-F 1 "GND" V 9905 4372 50  0000 R CNN
-F 2 "" H 9900 4500 50  0001 C CNN
-F 3 "" H 9900 4500 50  0001 C CNN
-	1    9900 4500
-	0    1    1    0
-$EndComp
-Wire Wire Line
-	9750 4600 9950 4600
+P 9950 4200
+F 0 "#PWR033" H 9950 3950 50  0001 C CNN
+F 1 "GND" V 9955 4072 50  0000 R CNN
+F 2 "" H 9950 4200 50  0001 C CNN
+F 3 "" H 9950 4200 50  0001 C CNN
+	1    9950 4200
+	0    1    1    0
+$EndComp
+Wire Wire Line
+	9800 4300 10000 4300
 $Comp
 L EXTENSION:74AHCV541ABQX IC1
@@
 Text GLabel 8600 2050 2    50   Input ~ 0
 YLED1
-Wire Wire Line
-	8600 1550 8550 1550
 Text GLabel 8600 1950 2    50   Input ~ 0
 YLED2
@@
 GLED2
 Wire Wire Line
-	8600 1650 8550 1650
-Wire Wire Line
 	8600 1750 8550 1750
 Wire Wire Line
 	8600 1850 8550 1850
-Text GLabel 8600 1650 2    50   Input ~ 0
-BUZZ1
-Text GLabel 8600 1550 2    50   Input ~ 0
-BUZZ2
 Wire Wire Line
 	8600 2050 8550 2050
@@
 Wire Wire Line
 	8150 800  8150 850
-Text GLabel 7500 1550 0    50   Input ~ 0
-TBUZZ1
-Text GLabel 7500 1450 0    50   Input ~ 0
-TBUZZ2
 Wire Wire Line
 	7500 1950 7550 1950
@@
 Wire Wire Line
 	7500 1650 7550 1650
-Wire Wire Line
-	7500 1550 7550 1550
-Wire Wire Line
-	7500 1450 7550 1450
 $Comp
 L power:GND #PWR022
@@
 	1050 3050 1100 3050
 Wire Wire Line
-	10200 5050 10200 5100
-Wire Wire Line
 	8350 5250 8700 5250
 Wire Wire Line
@@
 VIN
 Text GLabel 1050 1650 0    50   Input ~ 0
-TBUZZ1
-Text GLabel 1050 1750 0    50   Input ~ 0
-TBUZZ2
+PDECT1
 Wire Wire Line
 	1050 1750 1100 1750
@@
 Text Notes 5400 6750 0    50   ~ 0
 Accelerometer\nCommunicate I2C\n
+Text GLabel 7450 1450 0    50   Input ~ 0
+INFREE3
+Wire Wire Line
+	7450 1450 7550 1450
+Text GLabel 7450 1550 0    50   Input ~ 0
+INFREE4
+Wire Wire Line
+	7450 1550 7550 1550
+Text GLabel 8650 1550 2    50   Input ~ 0
+OUTFREE3
+Text GLabel 8650 1650 2    50   Input ~ 0
+OUTFREE4
+Wire Wire Line
+	8550 1550 8650 1550
+Wire Wire Line
+	8550 1650 8650 1650
+Text GLabel 1050 1750 0    50   Input ~ 0
+PDECT2
+$Comp
+L EXTENSION:505567-0671 J5
+U 1 1 61AEC270
+P 10250 4850
+F 0 "J5" H 10700 5115 50  0000 C CNN
+F 1 "EXTOUT" H 10700 5024 50  0000 C CNN
+F 2 "EXTENSION:5055670671" H 11000 4950 50  0001 L CNN
+F 3 "https://componentsearchengine.com/Datasheets/1/505567-0671.pdf" H 11000 4850 50  0001 L CNN
+F 4 "Molex Micro-Lock PLUS 505567, 1.25mm Pitch, 6 Way, 1 Row, Right Angle PCB Header, Surface Mount" H 11000 4750 50  0001 L CNN "Description"
+F 5 "4.2" H 11000 4650 50  0001 L CNN "Height"
+F 6 "538-505567-0671" H 11000 4550 50  0001 L CNN "Mouser Part Number"
+F 7 "https://www.mouser.co.uk/ProductDetail/Molex/505567-0671?qs=gt1LBUVyoHmQuimOt9l14w%3D%3D" H 11000 4450 50  0001 L CNN "Mouser Price/Stock"
+F 8 "Molex" H 11000 4350 50  0001 L CNN "Manufacturer_Name"
+F 9 "505567-0671" H 11000 4250 50  0001 L CNN "Manufacturer_Part_Number"
+	1    10250 4850
+	1    0    0    -1
+$EndComp
+$Comp
+L power:GND #PWR0101
+U 1 1 61AED9C0
+P 9900 4950
+F 0 "#PWR0101" H 9900 4700 50  0001 C CNN
+F 1 "GND" V 9905 4822 50  0000 R CNN
+F 2 "" H 9900 4950 50  0001 C CNN
+F 3 "" H 9900 4950 50  0001 C CNN
+	1    9900 4950
+	0    1    1    0
+$EndComp
+Text GLabel 10200 5050 0    50   Input ~ 0
+PDECT1
+Text GLabel 10200 5150 0    50   Input ~ 0
+PDECT2
+Text GLabel 10200 5250 0    50   Input ~ 0
+OPYRO1
+Text GLabel 10200 5350 0    50   Input ~ 0
+OPYRO2
+Wire Wire Line
+	10200 5250 10250 5250
+Wire Wire Line
+	10200 5150 10250 5150
+Wire Wire Line
+	10200 5050 10250 5050
+$Comp
+L power:+3.3V #PWR0102
+U 1 1 61B21118
+P 10200 4850
+F 0 "#PWR0102" H 10200 4700 50  0001 C CNN
+F 1 "+3.3V" V 10215 4978 50  0000 L CNN
+F 2 "" H 10200 4850 50  0001 C CNN
+F 3 "" H 10200 4850 50  0001 C CNN
+	1    10200 4850
+	0    -1   -1   0
+$EndComp
+Wire Wire Line
+	9900 4950 10250 4950
+Wire Wire Line
+	10200 4850 10250 4850
+Wire Wire Line
+	10200 5350 10250 5350
 $EndSCHEMATC

Commit message: a
Other:
- note added: "Mikro Lock Connectors\n"
- note removed: "Les connecteurs Mikro Lock"
Changed lines of the file:
@@
 Both Iacoboard and Teensy can fire pyros\nDiodes just to prevent them firing in each other
 Text Notes 9200 5900 0    50   ~ 0
-Les connecteurs Mikro Lock
+Mikro Lock Connectors\n
 Text Notes 10300 2750 0    50   ~ 0
 LEDs debug

Commit message: aaa
Parts:
- removed R4: 1k, Resistor_SMD:R_0603_1608Metric, symbol Device:R
- added D10: DIODE, Diode_SMD:D_0603_1608Metric, symbol Simulation_SPICE:DIODE
- added R12, R6: 3.3K, Resistor_SMD:R_0603_1608Metric, symbol Device:R
- C1: value 22pF -> 100nF
- R2, R3: value 10k -> 3.3K
Connections:
- net +3V3: now also D10.2 (K), R12.1, R6.1
- net Accel_SCL: now also R6.2
- net Accel_SDA: now also R12.2
- net Buzzer: now also D10.1 (A)
Changed lines of the file:
@@
 P 2650 4600
 F 0 "C1" H 2765 4646 50  0000 L CNN
-F 1 "22pF" H 2765 4555 50  0000 L CNN
+F 1 "100nF" H 2765 4555 50  0000 L CNN
 F 2 "Capacitor_SMD:C_0603_1608Metric" H 2688 4450 50  0001 C CNN
 F 3 "~" H 2650 4600 50  0001 C CNN
@@
 P 6050 950
 F 0 "R2" V 5843 950 50  0000 C CNN
-F 1 "10k" V 5934 950 50  0000 C CNN
+F 1 "3.3K" V 5934 950 50  0000 C CNN
 F 2 "Resistor_SMD:R_0603_1608Metric" V 5980 950 50  0001 C CNN
 F 3 "~" H 6050 950 50  0001 C CNN
@@
 P 6400 950
 F 0 "R3" V 6193 950 50  0000 C CNN
-F 1 "10k" V 6284 950 50  0000 C CNN
+F 1 "3.3K" V 6284 950 50  0000 C CNN
 F 2 "Resistor_SMD:R_0603_1608Metric" V 6330 950 50  0001 C CNN
 F 3 "~" H 6400 950 50  0001 C CNN
@@
 Wire Wire Line
 	4800 7200 4800 7150
-Wire Wire Line
-	4600 7200 4600 7150
-Text GLabel 4600 7200 0    50   Input ~ 0
+Text GLabel 4400 7200 0    50   Input ~ 0
 Accel_SDA
-Wire Wire Line
-	3850 6050 3900 6050
-Text GLabel 3850 6050 0    50   Input ~ 0
+Text GLabel 3600 6050 0    50   Input ~ 0
 Accel_SCL
 Wire Wire Line
@@
 Wire Wire Line
 	7500 2150 7550 2150
-Connection ~ 4850 3350
-Connection ~ 4850 3050
-Wire Wire Line
-	4750 3050 4850 3050
 Text GLabel 4850 3450 3    50   Input ~ 0
 Buzzer
@@
 	5100 3250 5050 3250
 Wire Wire Line
-	5050 3050 4850 3050
-Wire Wire Line
 	5050 3150 5050 3050
 Wire Wire Line
 	5100 3150 5050 3150
-$Comp
-L Device:R R4
-U 1 1 6181218E
-P 4850 3200
-F 0 "R4" H 4920 3246 50  0000 L CNN
-F 1 "1k" H 4920 3155 50  0000 L CNN
-F 2 "Resistor_SMD:R_0603_1608Metric" V 4780 3200 50  0001 C CNN
-F 3 "~" H 4850 3200 50  0001 C CNN
-	1    4850 3200
-	1    0    0    -1
-$EndComp
 $Comp
 L SamacSys_Parts:PS1240P02CT3 LS1
@@
 Wire Wire Line
 	10200 5350 10250 5350
+$Comp
+L Device:R R6
+U 1 1 619C990D
+P 3650 6300
+F 0 "R6" V 3443 6300 50  0000 C CNN
+F 1 "3.3K" V 3534 6300 50  0000 C CNN
+F 2 "Resistor_SMD:R_0603_1608Metric" V 3580 6300 50  0001 C CNN
+F 3 "~" H 3650 6300 50  0001 C CNN
+	1    3650 6300
+	-1   0    0    1
+$EndComp
+Wire Wire Line
+	3650 6150 3650 6050
+Wire Wire Line
+	3650 6050 3600 6050
+Wire Wire Line
+	3650 6050 3900 6050
+Connection ~ 3650 6050
+$Comp
+L power:+3.3V #PWR0103
+U 1 1 619DF704
+P 3650 6500
+F 0 "#PWR0103" H 3650 6350 50  0001 C CNN
+F 1 "+3.3V" V 3665 6628 50  0000 L CNN
+F 2 "" H 3650 6500 50  0001 C CNN
+F 3 "" H 3650 6500 50  0001 C CNN
+	1    3650 6500
+	-1   0    0    1
+$EndComp
+Wire Wire Line
+	3650 6500 3650 6450
+$Comp
+L Device:R R12
+U 1 1 619EA19E
+P 4400 7400
+F 0 "R12" V 4193 7400 50  0000 C CNN
+F 1 "3.3K" V 4284 7400 50  0000 C CNN
+F 2 "Resistor_SMD:R_0603_1608Metric" V 4330 7400 50  0001 C CNN
+F 3 "~" H 4400 7400 50  0001 C CNN
+	1    4400 7400
+	0    -1   -1   0
+$EndComp
+Wire Wire Line
+	4550 7400 4600 7400
+Wire Wire Line
+	4600 7150 4600 7200
+Wire Wire Line
+	4600 7200 4400 7200
+Connection ~ 4600 7200
+Wire Wire Line
+	4600 7200 4600 7400
+$Comp
+L power:+3.3V #PWR0104
+U 1 1 619FF8A5
+P 4200 7400
+F 0 "#PWR0104" H 4200 7250 50  0001 C CNN
+F 1 "+3.3V" V 4215 7528 50  0000 L CNN
+F 2 "" H 4200 7400 50  0001 C CNN
+F 3 "" H 4200 7400 50  0001 C CNN
+	1    4200 7400
+	0    -1   -1   0
+$EndComp
+Wire Wire Line
+	4200 7400 4250 7400
+$Comp
+L Simulation_SPICE:DIODE D10
+U 1 1 61A0E772
+P 4850 3200
+F 0 "D10" H 4850 3417 50  0000 C CNN
+F 1 "DIODE" H 4850 3326 50  0000 C CNN
+F 2 "Diode_SMD:D_0603_1608Metric" H 4850 3200 50  0001 C CNN
+F 3 "~" H 4850 3200 50  0001 C CNN
+F 4 "Y" H 4850 3200 50  0001 L CNN "Spice_Netlist_Enabled"
+F 5 "D" H 4850 3200 50  0001 L CNN "Spice_Primitive"
+	1    4850 3200
+	0    -1   -1   0
+$EndComp
+Wire Wire Line
+	4750 3050 4850 3050
+Connection ~ 4850 3350
+Connection ~ 4850 3050
+Wire Wire Line
+	4850 3050 5050 3050
 $EndSCHEMATC

Commit message: last changes
Parts:
- removed R12, R6: 3.3K, Resistor_SMD:R_0603_1608Metric, symbol Device:R
Connections:
- net Accel_SCL: now also IC2.8 (SCLK), R2.1
- net Accel_SDA: now also IC2.7 (SDI/SDA), R3.1
- removed net Baro_SCLK: IC2.8 (SCLK), R2.1, U2.23 (16_A2_RX4_SCL1)
- removed net Baro_SDA: IC2.7 (SDI/SDA), R3.1, U2.24 (17_A3_TX4_SDA1)
Changed lines of the file:
@@
 Connection ~ 4250 1450
 Text GLabel 6450 1200 2    50   Input ~ 0
-Baro_SDA
+Accel_SDA
 Text GLabel 5900 1050 1    50   Input ~ 0
-Baro_SCLK
+Accel_SCL
 $Comp
 L EXTENSION:COM-15809 U1
@@
 	5850 1300 5850 1400
 Connection ~ 5850 1400
-Text GLabel 1050 3250 0    50   Input ~ 0
-Baro_SDA
-Wire Wire Line
-	1050 3250 1100 3250
-Text GLabel 1050 3150 0    50   Input ~ 0
-Baro_SCLK
-Wire Wire Line
-	1050 3150 1100 3150
 $Comp
 L power:GND #PWR014
@@
 Wire Wire Line
 	10200 5350 10250 5350
-$Comp
-L Device:R R6
-U 1 1 619C990D
-P 3650 6300
-F 0 "R6" V 3443 6300 50  0000 C CNN
-F 1 "3.3K" V 3534 6300 50  0000 C CNN
-F 2 "Resistor_SMD:R_0603_1608Metric" V 3580 6300 50  0001 C CNN
-F 3 "~" H 3650 6300 50  0001 C CNN
-	1    3650 6300
-	-1   0    0    1
-$EndComp
-Wire Wire Line
-	3650 6150 3650 6050
-Wire Wire Line
-	3650 6050 3600 6050
-Wire Wire Line
-	3650 6050 3900 6050
-Connection ~ 3650 6050
-$Comp
-L power:+3.3V #PWR0103
-U 1 1 619DF704
-P 3650 6500
-F 0 "#PWR0103" H 3650 6350 50  0001 C CNN
-F 1 "+3.3V" V 3665 6628 50  0000 L CNN
-F 2 "" H 3650 6500 50  0001 C CNN
-F 3 "" H 3650 6500 50  0001 C CNN
-	1    3650 6500
-	-1   0    0    1
-$EndComp
-Wire Wire Line
-	3650 6500 3650 6450
-$Comp
-L Device:R R12
-U 1 1 619EA19E
-P 4400 7400
-F 0 "R12" V 4193 7400 50  0000 C CNN
-F 1 "3.3K" V 4284 7400 50  0000 C CNN
-F 2 "Resistor_SMD:R_0603_1608Metric" V 4330 7400 50  0001 C CNN
-F 3 "~" H 4400 7400 50  0001 C CNN
-	1    4400 7400
-	0    -1   -1   0
-$EndComp
-Wire Wire Line
-	4550 7400 4600 7400
 Wire Wire Line
 	4600 7150 4600 7200
 Wire Wire Line
 	4600 7200 4400 7200
-Connection ~ 4600 7200
-Wire Wire Line
-	4600 7200 4600 7400
-$Comp
-L power:+3.3V #PWR0104
-U 1 1 619FF8A5
-P 4200 7400
-F 0 "#PWR0104" H 4200 7250 50  0001 C CNN
-F 1 "+3.3V" V 4215 7528 50  0000 L CNN
-F 2 "" H 4200 7400 50  0001 C CNN
-F 3 "" H 4200 7400 50  0001 C CNN
-	1    4200 7400
-	0    -1   -1   0
-$EndComp
-Wire Wire Line
-	4200 7400 4250 7400
 $Comp
 L Simulation_SPICE:DIODE D10
@@
 Wire Wire Line
 	4850 3050 5050 3050
+Wire Wire Line
+	3600 6050 3900 6050
 $EndSCHEMATC
