File: CLIP_HOSTBOARD/CLIP_HOSTBOARD.kicad_pcb (KiCad board)
At the start: 2 copper layers, 50 x 20.4 mm, 7 parts, among them J1 505567-0671, J2 1x2_header, J3 1x5_header, U1 Buffer

Commit message: duh
Routing:
- net GND: vias 3 -> 4
Changed lines of the file:
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@@
   (general
     (thickness 1.6)
-    (drawings 6)
-    (tracks 103)
+    (drawings 8)
+    (tracks 104)
     (zones 0)
     (modules 7)
@@
     )
   )
+  (dimension 20.40128 (width 0.15) (layer Dwgs.User)
+    (gr_text "20.401 mm" (at 172.844435 90.697804 -89.99286656) (layer Dwgs.User)
+      (effects (font (size 1 1) (thickness 0.15)))
+    )
+    (feature1 (pts (xy 168.69664 80.49768) (xy 172.129586 80.497253)))
+    (feature2 (pts (xy 168.69918 100.89896) (xy 172.132126 100.898533)))
+    (crossbar (pts (xy 171.545705 100.898606) (xy 171.543165 80.497326)))
+    (arrow1a (pts (xy 171.543165 80.497326) (xy 172.129726 81.623757)))
+    (arrow1b (pts (xy 171.543165 80.497326) (xy 170.956885 81.623903)))
+    (arrow2a (pts (xy 171.545705 100.898606) (xy 172.131985 99.772029)))
+    (arrow2b (pts (xy 171.545705 100.898606) (xy 170.959144 99.772175)))
+  )
+  (dimension 49.999903 (width 0.15) (layer Dwgs.User)
+    (gr_text "50.000 mm" (at 143.700182 105.358283 359.9796256) (layer Dwgs.User)
+      (effects (font (size 1 1) (thickness 0.15)))
+    )
+    (feature1 (pts (xy 168.70172 100.9015) (xy 168.700386 104.653594)))
+    (feature2 (pts (xy 118.70182 100.88372) (xy 118.700486 104.635814)))
+    (crossbar (pts (xy 118.700694 104.049393) (xy 168.700594 104.067173)))
+    (arrow1a (pts (xy 168.700594 104.067173) (xy 167.573882 104.653193)))
+    (arrow1b (pts (xy 168.700594 104.067173) (xy 167.574299 103.480352)))
+    (arrow2a (pts (xy 118.700694 104.049393) (xy 119.826989 104.636214)))
+    (arrow2b (pts (xy 118.700694 104.049393) (xy 119.827406 103.463373)))
+  )
   (gr_text "William\nCottier" (at 142.73022 82.296) (layer B.SilkS)
     (effects (font (size 0.5 0.5) (thickness 0.1)) (justify mirror))
@@
   (segment (start 148.0699 96.56572) (end 148.06482 96.56064) (width 0.25) (layer F.Cu) (net 4))
   (segment (start 149.53996 96.56572) (end 148.0699 96.56572) (width 0.25) (layer F.Cu) (net 4))
+  (via (at 144.61236 82.69732) (size 0.8) (drill 0.4) (layers F.Cu B.Cu) (net 4))
   (segment (start 143.99212 90.66538) (end 143.99212 87.092) (width 0.25) (layer F.Cu) (net 5))
   (segment (start 144.7627 86.32142) (end 144.7627 84.63514) (width 0.25) (layer F.Cu) (net 5))
