File: POWER_BOARD/POWER_BOARD.kicad_pcb (KiCad board)
At the start: 2 copper layers, 41 parts, among them IC1 ILQ30, J1 EXTIN, J2 ARM, J3 Pyro1, J4 Pyro2, J5 Servo2, J6 Servo1, J7 Batt, Q1 IRL40B212, Q2 IRL40B212, U1 SF-1206HH10M-2, U2 SF-1206HH10M-2, U3 AS358AP

Commit message: worked
Routing:
- net GND: track 0.00 -> 1.71 mm, vias 0 -> 7

Commit message: duh
Parts:
- removed J1: EXTIN, SamacSys_Parts:2828345
- added J8: EXTIN, EXTENSION:5055670571, F.Cu at (96.9, 94.8)
- D1, D2, D3, D4, D5: footprint digikey-footprints:LED_2-SMD_No_Lead_1.7x0.8mm -> KRTEK_V2:LED_2-SMD_No_Lead_1.7x0.8mm
- IC1: footprint SamacSys_Parts:DIP762W60P254L2030H430Q16N -> KRTEK_V2:DIP762W60P254L2030H430Q16N
- J2, J3, J4, J5, J6, J7: footprint SamacSys_Parts:282834-2_1 -> KRTEK_V2:282834-2_1
- PS1: footprint SamacSys_Parts:RPM5060 -> KRTEK_V2:RPM5060
- Q1, Q2: footprint SamacSys_Parts:TO254P483X1016X1994-3P -> KRTEK_V2:TO254P483X1016X1994-3P
- R9: value 66k -> 68k
Routing:
- net PYRO1IN: track 26.1 -> 6.95 mm
- net BUZZ1IN: track 25.2 -> 13.5 mm
- net BUZZ2IN: track 16.2 -> 11.1 mm
- net GNDIN: track 22.7 -> 20.6 mm
- net PYRO2IN: track 11.9 -> 9.93 mm

Commit message: Worked again
Connections:
- IC1 pad 12: BUZZ1IN -> BUZZ2IN
- IC1 pad 9: BUZZ2IN -> BUZZ1IN
Routing:
- net BUZZ2IN: track 11.1 -> 13.5 mm
- net BUZZ1IN: track 13.5 -> 11.1 mm

Commit message: t
Parts:
- removed J8: EXTIN, EXTENSION:5055670571
- added J9: 505567-0671, EXTENSION:5055670671, F.Cu at (97.3, 95.0)
- R2, R3: value 500 -> 510
Connections:
- IC1 pad 10: GNDIN -> 3V3IN
- IC1 pad 11: GNDIN -> 3V3IN
- IC1 pad 12: BUZZ2IN -> PDECT2IN
- IC1 pad 9: BUZZ1IN -> PDECT1IN
Routing:
- net 3V3IN: track 0.00 -> 22.9 mm, vias 0 -> 1
- net PDECT1IN: track 0.00 -> 17.7 mm, vias 0 -> 1
- net PDECT2IN: track 0.00 -> 16.3 mm, vias 0 -> 1
- net PYRO1IN: track 6.95 -> 21.2 mm
- net BUZZ2IN: track 13.5 -> 0.00 mm
- net BUZZ1IN: track 11.1 -> 0.00 mm
- net GNDIN: track 20.6 -> 12.4 mm
- net PYRO2IN: track 9.93 -> 11.0 mm

Commit message: aaa
Parts:
- J9: value 505567-0671 -> EXTIN
Connections:
- J6 pad 2: VINSERVO1 -> VINSERVO2
- PS1 pad A5: VINSERVO1 -> VINSERVO2
- PS1 pad D1: VCC -> Net-(PS1-PadD1)
Routing:
- net VINSERVO2: track 8.73 -> 16.9 mm
- net VINSERVO1: track 5.85 -> 0.00 mm
- net VCC: track 82.1 -> 81.1 mm

Commit message: last changes
Routing:
- net GND: track 1.71 -> 45.2 mm
Other:
- board outline added: 57 x 30 mm
- board text added: "ERT Wildhorn"
- board text added: "William Cottier"
Changed lines of the file:
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@@
   (general
     (thickness 1.6)
-    (drawings 5)
-    (tracks 268)
+    (drawings 11)
+    (tracks 282)
     (zones 0)
     (modules 41)
@@
     )
   )
+  (gr_line (start 95 80) (end 95 110) (layer Edge.Cuts) (width 0.15))
+  (gr_line (start 95 110) (end 152 110) (layer Edge.Cuts) (width 0.15))
+  (gr_line (start 152 80) (end 152 110) (layer Edge.Cuts) (width 0.15))
+  (gr_line (start 95 80) (end 152 80) (layer Edge.Cuts) (width 0.15))
+  (gr_text "ERT\nWildhorn" (at 129.07924 82.04346) (layer F.SilkS)
+    (effects (font (size 1 1) (thickness 0.15)))
+  )
+  (gr_text "William\nCottier" (at 125.3429 102.24408) (layer B.SilkS)
+    (effects (font (size 0.5 0.5) (thickness 0.1)) (justify mirror))
+  )
   (gr_text "KRTEK_V2\nR01\nPOWER BOARD" (at 128.3782 105.9474) (layer F.SilkS)
     (effects (font (size 1 1) (thickness 0.125)))
@@
   (segment (start 113.1114 108.0824) (end 112.427 108.0824) (width 0.25) (layer F.Cu) (net 2))
   (segment (start 113.4938 107.7) (end 113.1114 108.0824) (width 0.25) (layer F.Cu) (net 2))
+  (segment (start 119.7088 91.3718) (end 121.9988 93.6618) (width 1.25) (layer F.Cu) (net 2))
+  (segment (start 119.7088 93.6618) (end 121.9988 91.3718) (width 1.25) (layer F.Cu) (net 2))
+  (segment (start 121.9988 91.3718) (end 124.2888 93.6618) (width 1.25) (layer F.Cu) (net 2))
+  (segment (start 121.9988 93.6618) (end 124.2888 91.3718) (width 1.25) (layer F.Cu) (net 2))
+  (segment (start 121.9988 93.6618) (end 119.7088 95.9518) (width 1.25) (layer F.Cu) (net 2))
+  (segment (start 119.7088 93.6618) (end 121.9988 95.9518) (width 1.25) (layer F.Cu) (net 2))
+  (segment (start 119.7088 95.9518) (end 117.4188 93.6618) (width 1.25) (layer F.Cu) (net 2))
+  (segment (start 117.4188 95.9518) (end 119.7088 93.6618) (width 1.25) (layer F.Cu) (net 2))
+  (segment (start 117.4188 93.6618) (end 115.1288 91.3718) (width 1.25) (layer F.Cu) (net 2))
+  (segment (start 115.1288 93.6618) (end 117.4188 91.3718) (width 1.25) (layer F.Cu) (net 2))
+  (segment (start 117.4188 91.3718) (end 119.7088 93.6618) (width 1.25) (layer F.Cu) (net 2))
+  (segment (start 117.4188 93.6618) (end 119.7088 91.3718) (width 1.25) (layer F.Cu) (net 2))
+  (segment (start 117.4188 98.2418) (end 117.4188 95.9518) (width 1.25) (layer F.Cu) (net 2))
+  (segment (start 121.9988 89.0818) (end 121.9988 91.3718) (width 1.25) (layer F.Cu) (net 2))
   (segment (start 107.8296 106.5824) (end 107.8804 106.5316) (width 0.25) (layer F.Cu) (net 3))
   (segment (start 105.5944 106.5824) (end 107.8296 106.5824) (width 0.25) (layer F.Cu) (net 3))
@@
   (segment (start 98.081521 93.770199) (end 109.923001 93.770199) (width 0.25) (layer B.Cu) (net 32))
   (segment (start 97.51212 94.3396) (end 98.081521 93.770199) (width 0.25) (layer B.Cu) (net 32))
+  (zone (net 2) (net_name GND) (layer B.Cu) (hatch edge 0.508)
+    (connect_pads (clearance 0.508))
+    (min_thickness 0.254)
+    (fill yes (arc_segments 32) (thermal_gap 0.508) (thermal_bridge_width 0.508))
+    (polygon
+      (pts
+        (xy 152.02814 110.00378) (xy 95.02038 109.98854) (xy 95.02038 79.99876) (xy 95.06356 79.99876) (xy 152.0002 79.97082)
+      )
+    )
+  )
   (zone (net 2) (net_name GND) (layer F.Cu) (hatch edge 0.508)
     (connect_pads (clearance 0.508))
@@
     (polygon
       (pts
-        (xy 153.18765 110.89405) (xy 94.0882 110.748) (xy 94.0882 79.125) (xy 152.7241 78.6297)
+        (xy 152.05862 109.98854) (xy 95.02038 110.01648) (xy 94.9899 79.97082) (xy 152.0256 79.98352)
       )
     )
     (polygon
       (pts
-        (xy 92.564164 78.997799) (xy 92.5134 78.998) (xy 92.5642 78.9726)
+        (xy 94.94926 80.04956) (xy 94.94926 80.05718)
       )
     )
-  )
-  (zone (net 2) (net_name GND) (layer B.Cu) (hatch edge 0.508)
-    (connect_pads (clearance 0.508))
-    (min_thickness 0.254)
-    (fill yes (arc_segments 32) (thermal_gap 0.508) (thermal_bridge_width 0.508))
-    (polygon
-      (pts
-        (xy 152.7749 110.5702) (xy 94.10725 110.6083) (xy 93.96755 78.8329) (xy 94.0882 78.744) (xy 152.559 79.1504)
-      )
-    )
