File: POWER_BOARD/POWER_BOARD.kicad_pcb (KiCad board)
At the start: 2 copper layers, 57 x 30 mm, 41 parts, among them IC1 ILQ30, J2 ARM, J3 Pyro1, J4 Pyro2, J5 Servo2, J6 Servo1, J7 Batt, J9 EXTIN, Q1 IRL40B212, Q2 IRL40B212, U1 SF-1206HH10M-2, U2 SF-1206HH10M-2, U3 AS358AP

Commit message: duh
Connections:
- J9 pad 1: PYRO1IN -> PYRO2IN
- J9 pad 2: PYRO2IN -> PYRO1IN
Routing:
- net PYRO1IN: track 21.2 -> 24.6 mm, vias 0 -> 2
- net PYRO2IN: track 11.0 -> 12.5 mm
Other:
- rule via_min_size: 0.4 -> 0.3
Changed lines of the file:
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@@
   (general
     (thickness 1.6)
-    (drawings 11)
-    (tracks 282)
+    (drawings 13)
+    (tracks 289)
     (zones 0)
     (modules 41)
@@
     (via_size 0.8)
     (via_drill 0.4)
-    (via_min_size 0.4)
+    (via_min_size 0.3)
     (via_min_drill 0.3)
     (uvia_size 0.3)
@@
     (fp_arc (start -4 2.15) (end -4 2.25) (angle -180) (layer F.SilkS) (width 0.2))
     (pad 1 smd rect (at -3.125 1.6 90) (size 0.8 1.2) (layers F.Cu F.Paste F.Mask)
+      (net 9 PYRO2IN))
+    (pad 2 smd rect (at -1.875 1.6 90) (size 0.8 1.2) (layers F.Cu F.Paste F.Mask)
       (net 7 PYRO1IN))
-    (pad 2 smd rect (at -1.875 1.6 90) (size 0.8 1.2) (layers F.Cu F.Paste F.Mask)
-      (net 9 PYRO2IN))
     (pad 3 smd rect (at -0.625 1.6 90) (size 0.8 1.2) (layers F.Cu F.Paste F.Mask)
       (net 30 PDECT1IN))
@@
       (rotate (xyz 0 0 0))
     )
+  )
+  (dimension 30.00378 (width 0.15) (layer Dwgs.User)
+    (gr_text "30.004 mm" (at 80.315984 95.000677 89.99526415) (layer Dwgs.User)
+      (effects (font (size 1 1) (thickness 0.15)))
+    )
+    (feature1 (pts (xy 95 80) (xy 81.030803 79.998845)))
+    (feature2 (pts (xy 94.99752 110.00378) (xy 81.028323 110.002625)))
+    (crossbar (pts (xy 81.614744 110.002674) (xy 81.617224 79.998894)))
+    (arrow1a (pts (xy 81.617224 79.998894) (xy 82.203552 81.125446)))
+    (arrow1b (pts (xy 81.617224 79.998894) (xy 81.03071 81.125349)))
+    (arrow2a (pts (xy 81.614744 110.002674) (xy 82.201258 108.876219)))
+    (arrow2b (pts (xy 81.614744 110.002674) (xy 81.028416 108.876122)))
+  )
+  (dimension 57.00522 (width 0.15) (layer Dwgs.User)
+    (gr_text "57.005 mm" (at 123.496692 120.081528 359.9948941) (layer Dwgs.User)
+      (effects (font (size 1 1) (thickness 0.15)))
+    )
+    (feature1 (pts (xy 152.0002 110.00632) (xy 151.999366 119.370489)))
+    (feature2 (pts (xy 94.99498 110.00124) (xy 94.994146 119.365409)))
+    (crossbar (pts (xy 94.994198 118.778988) (xy 151.999418 118.784068)))
+    (arrow1a (pts (xy 151.999418 118.784068) (xy 150.872862 119.370388)))
+    (arrow1b (pts (xy 151.999418 118.784068) (xy 150.872967 118.197547)))
+    (arrow2a (pts (xy 94.994198 118.778988) (xy 96.120649 119.365509)))
+    (arrow2b (pts (xy 94.994198 118.778988) (xy 96.120754 118.192668)))
   )
   (gr_line (start 95 80) (end 95 110) (layer Edge.Cuts) (width 0.15))
@@
   (segment (start 114.5352 106.5824) (end 114.6114 106.5062) (width 0.25) (layer F.Cu) (net 6))
   (segment (start 112.427 106.5824) (end 114.5352 106.5824) (width 0.25) (layer F.Cu) (net 6))
+  (via (at 97.49434 96.82118) (size 0.8) (drill 0.4) (layers F.Cu B.Cu) (net 7))
   (segment (start 103.4608 81.9952) (end 103.918 81.9952) (width 0.25) (layer F.Cu) (net 7))
-  (segment (start 99.74114 98.09198) (end 102.12222 95.7109) (width 0.25) (layer F.Cu) (net 7))
-  (segment (start 98.89114 98.09198) (end 99.74114 98.09198) (width 0.25) (layer F.Cu) (net 7))
   (segment (start 102.12222 95.7109) (end 102.12222 92.0155) (width 0.25) (layer F.Cu) (net 7))
   (segment (start 102.12222 92.0155) (end 103.26014 90.87758) (width 0.25) (layer F.Cu) (net 7))
@@
   (segment (start 105.41914 83.49634) (end 103.918 81.9952) (width 0.25) (layer F.Cu) (net 7))
   (segment (start 105.41914 90.09272) (end 105.41914 83.49634) (width 0.25) (layer F.Cu) (net 7))
+  (segment (start 99.226142 96.84198) (end 98.89114 96.84198) (width 0.25) (layer F.Cu) (net 7))
+  (segment (start 102.12222 95.7109) (end 102.12222 96.92024) (width 0.25) (layer F.Cu) (net 7))
+  (segment (start 102.12222 96.92024) (end 102.12222 96.92024) (width 0.25) (layer F.Cu) (net 7))
+  (via (at 102.12222 96.92024) (size 0.8) (drill 0.4) (layers F.Cu B.Cu) (net 7))
+  (segment (start 97.5934 96.92024) (end 97.49434 96.82118) (width 0.25) (layer B.Cu) (net 7))
+  (segment (start 102.12222 96.92024) (end 97.5934 96.92024) (width 0.25) (layer B.Cu) (net 7))
+  (segment (start 98.87034 96.82118) (end 98.89114 96.84198) (width 0.25) (layer F.Cu) (net 7))
+  (segment (start 97.49434 96.82118) (end 98.87034 96.82118) (width 0.25) (layer F.Cu) (net 7))
   (segment (start 103.918 84.5352) (end 103.918 87.0752) (width 0.25) (layer F.Cu) (net 8))
   (segment (start 103.918 87.0752) (end 101.76916 87.0752) (width 0.25) (layer F.Cu) (net 8))
@@
   (segment (start 100.47884 92.35428) (end 99.74114 93.09198) (width 0.25) (layer F.Cu) (net 8))
   (segment (start 100.47884 88.36552) (end 100.47884 92.35428) (width 0.25) (layer F.Cu) (net 8))
+  (segment (start 99.74114 98.09198) (end 98.89114 98.09198) (width 0.25) (layer F.Cu) (net 9))
+  (segment (start 100.92885 96.90427) (end 99.74114 98.09198) (width 0.25) (layer F.Cu) (net 9))
+  (segment (start 100.92885 90.06435) (end 100.92885 96.90427) (width 0.25) (layer F.Cu) (net 9))
+  (segment (start 101.378 89.6152) (end 100.92885 90.06435) (width 0.25) (layer F.Cu) (net 9))
   (segment (start 103.918 89.6152) (end 101.378 89.6152) (width 0.25) (layer F.Cu) (net 9))
-  (segment (start 99.226142 96.84198) (end 98.89114 96.84198) (width 0.25) (layer F.Cu) (net 9))
-  (segment (start 100.92885 95.139272) (end 99.226142 96.84198) (width 0.25) (layer F.Cu) (net 9))
-  (segment (start 100.92885 90.06435) (end 100.92885 95.139272) (width 0.25) (layer F.Cu) (net 9))
-  (segment (start 101.378 89.6152) (end 100.92885 90.06435) (width 0.25) (layer F.Cu) (net 9))
   (segment (start 132.3132 103.7366) (end 132.111 103.5344) (width 0.25) (layer B.Cu) (net 10))
   (segment (start 135.414 103.7366) (end 132.3132 103.7366) (width 0.25) (layer B.Cu) (net 10))

Commit message: last commit
Parts:
- removed G***: LOGO, KRTEK_V2:b_smol_KRTEK_LOGO
- removed the REF** at (148.5, 106.5)
- removed the REF** at (98.6, 83.4)
- removed the REF** at (98.6, 106.4)
- removed U3: AS358AP, KRTEK_V2:AS358AP-PDIP-8
- added Q3: NX3020NAK,215, Package_TO_SOT_SMD:SOT-23, B.Cu at (130.1, 93.0)
- added Q4: NX3020NAK,215, Package_TO_SOT_SMD:SOT-23, B.Cu at (130.0, 99.6)
- added REF**: MountingHole_3.2mm_M3, MountingHole:MountingHole_3.2mm_M3, F.Cu at (98.6, 106.4)
- added REF**: MountingHole_3.2mm_M3, MountingHole:MountingHole_3.2mm_M3, F.Cu at (98.6, 83.6)
- added REF**: MountingHole_3.2mm_M3, MountingHole:MountingHole_3.2mm_M3, F.Cu at (148.4, 106.4)
- R10, R8: value 34k -> 500
- R11: value 66k -> 215k
- R14, R15: value 10k -> 740
- R16, R17: value 10k -> 740; moved to F.Cu
- R9: value 68k -> 215k
- moved R14 28.8 mm to (107.8, 94.8), turned to 0 degrees
- moved R15 24.1 mm to (108.0, 97.6), turned to 0 degrees
- moved R9 17.1 mm to (133.0, 90.2), turned to -90 degrees
- moved R8 14.3 mm to (133.8, 92.8)
- moved R17 13.8 mm to (124.6, 106.0), turned to 180 degrees
- moved R10 12.1 mm to (133.6, 99.6)
- moved R11 8.98 mm to (133.6, 97.6), turned to 180 degrees
- moved R16 4.89 mm to (128.2, 96.8)
Connections:
- IC1 pad 12: PDECT2IN -> Net-(IC1-Pad12)
- IC1 pad 13: VCC -> OPTO2
- IC1 pad 14: OPTO2 -> VCC
- IC1 pad 15: OPTO1 -> VCC
- IC1 pad 16: VCC -> OPTO1
- IC1 pad 5: BUZZ1 -> VCC
- IC1 pad 6: GND -> BUZZ1
- IC1 pad 7: GND -> BUZZ2
- IC1 pad 8: BUZZ2 -> VCC
- IC1 pad 9: PDECT1IN -> Net-(IC1-Pad9)
- J3 pad 1: PYRO1 -> AMP1
- J4 pad 1: PYRO2 -> AMP2
- J9 pad MP1: Net-(J9-PadMP1) -> unconnected-(J9-PadMP1)
- J9 pad MP2: Net-(J9-PadMP2) -> unconnected-(J9-PadMP2)
- PS1 pad B2: GND -> unconnected-(PS1-PadB2)
- PS1 pad B3: GND -> unconnected-(PS1-PadB3)
- PS1 pad D1: Net-(PS1-PadD1) -> unconnected-(PS1-PadD1)
- PS1 pad D3: GND -> unconnected-(PS1-PadD3)
- PS1 pad D4: GND -> unconnected-(PS1-PadD4)
- PS1 pad E1: Net-(PS1-PadE1) -> unconnected-(PS1-PadE1)
- PS1 pad E2: Net-(PS1-PadE2) -> unconnected-(PS1-PadE2)
- Q1 pad 2: PYRO1 -> AMP1
- Q2 pad 2: PYRO2 -> AMP2
- R10 pad 1: AMP2 -> Net-(Q4-Pad1)
- R10 pad 2: PYRO2 -> AMP1
- R11 pad 2: AMP2 -> Net-(Q4-Pad1)
- R14 pad 1: Net-(R14-Pad1) -> PDECT2IN
- R14 pad 2: BUZZ1 -> Net-(IC1-Pad12)
- R15 pad 1: BUZZ1 -> PDECT1IN
- R15 pad 2: GND -> Net-(IC1-Pad9)
- R16 pad 1: BUZZ2 -> Net-(Q3-Pad3)
- R16 pad 2: GND -> BUZZ2
- R17 pad 2: BUZZ2 -> BUZZ1
- R6 pad 2: PYRO1 -> AMP1
- R7 pad 2: PYRO2 -> AMP2
- R8 pad 1: AMP1 -> Net-(Q3-Pad1)
- R8 pad 2: PYRO1 -> AMP2
- R9 pad 2: AMP1 -> Net-(Q3-Pad1)
Routing:
- net PYRO2: track 56.5 -> 0.00 mm, vias 3 -> 0
- net PYRO1: track 54.3 -> 0.00 mm, vias 1 -> 0
- net AMP1: track 17.2 -> 62.1 mm, vias 2 -> 1
- net AMP2: track 11.0 -> 51.4 mm, vias 0 -> 3
- net BUZZ1: track 58.4 -> 36.1 mm, vias 1 -> 0
- net VCC: track 81.1 -> 97.1 mm, vias 0 -> 2
- net OPTO2: track 37.1 -> 52.9 mm, vias 2 -> 3
- net GND: track 45.2 -> 57.4 mm, vias 7 -> 9
- net BUZZ2: track 54.0 -> 44.6 mm
- net Net-(R14-Pad1): track 6.45 -> 0.00 mm
- net PDECT1IN: track 17.7 -> 11.9 mm
- net PDECT2IN: track 16.3 -> 11.8 mm
- net Net-(Q3-Pad3): track 0.00 -> 4.28 mm, vias 0 -> 1
- net Net-(Q4-Pad3): track 4.13 -> 8.34 mm, vias 0 -> 1
- net Net-(Q4-Pad1): track 0.00 -> 4.21 mm
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Other:
- net class Default removed
