File: POWER_BOARD/POWER_BOARD.sch (KiCad schematic (older format))
At the start: 37 parts, among them IC1 ILQ30, J1 EXTIN, J2 ARM, J3 Pyro1, J4 Pyro2, J5 Servo2, J6 Servo1, J7 Batt, Q1 IRL40B212, Q2 IRL40B212, U1 SF-1206HH10M-2, U2 SF-1206HH10M-2, U3 AS358AP

Commit message: Update POWER_BOARD.sch
Parts:
- U1, U2: symbol KRTEK_V2:SF-1206HH10M-2 -> POWER_BOARD-rescue:SF-1206HH10M-2-KRTEK_V2
- U3: symbol KRTEK_V2:AS358AP -> POWER_BOARD-rescue:AS358AP-KRTEK_V2
Changed lines of the file:
@@
 	1850 2750 1850 2800
 $Comp
-L KRTEK_V2:AS358AP U3
+L POWER_BOARD-rescue:AS358AP-KRTEK_V2 U3
 U 1 1 617A35D3
 P 9400 1850
@@
 	4850 4600 4550 4600
 $Comp
-L KRTEK_V2:SF-1206HH10M-2 U1
+L POWER_BOARD-rescue:SF-1206HH10M-2-KRTEK_V2 U1
 U 1 1 6198B2D9
 P 4350 4100
@@
 $EndComp
 $Comp
-L KRTEK_V2:SF-1206HH10M-2 U2
+L POWER_BOARD-rescue:SF-1206HH10M-2-KRTEK_V2 U2
 U 1 1 6198C1F2
 P 4350 4550

Commit message: duh
Parts:
- added J8: EXTIN, EXTENSION:5055670571, symbol EXTENSION:505567-0571
Connections:
- net BUZZ1IN: now also J8.3
- net BUZZ2IN: now also J8.4
- net GNDIN: now also J8.5
- net PYRO1IN: now also J8.1
- net PYRO2IN: now also J8.2
Changed lines of the file:
@@
 Text GLabel 3650 7500 2    50   Input ~ 0
 PYRO2
-Wire Wire Line
-	5600 7400 5500 7400
 $Comp
 L power:VCC #PWR016
 U 1 1 61877079
-P 5600 7400
-F 0 "#PWR016" H 5600 7250 50  0001 C CNN
-F 1 "VCC" H 5615 7573 50  0000 C CNN
-F 2 "" H 5600 7400 50  0001 C CNN
-F 3 "" H 5600 7400 50  0001 C CNN
-	1    5600 7400
+P 5550 7400
+F 0 "#PWR016" H 5550 7250 50  0001 C CNN
+F 1 "VCC" H 5565 7573 50  0000 C CNN
+F 2 "" H 5550 7400 50  0001 C CNN
+F 3 "" H 5550 7400 50  0001 C CNN
+	1    5550 7400
 	0    1    1    0
 $EndComp
@@
 L power:GND #PWR017
 U 1 1 61877E3F
-P 5800 7500
-F 0 "#PWR017" H 5800 7250 50  0001 C CNN
-F 1 "GND" H 5805 7327 50  0000 C CNN
-F 2 "" H 5800 7500 50  0001 C CNN
-F 3 "" H 5800 7500 50  0001 C CNN
-	1    5800 7500
-	0    -1   -1   0
-$EndComp
-Wire Wire Line
-	5500 7500 5800 7500
+P 5500 7550
+F 0 "#PWR017" H 5500 7300 50  0001 C CNN
+F 1 "GND" H 5505 7377 50  0000 C CNN
+F 2 "" H 5500 7550 50  0001 C CNN
+F 3 "" H 5500 7550 50  0001 C CNN
+	1    5500 7550
+	1    0    0    -1
+$EndComp
 $Comp
 L SamacSys_Parts:RPM5.0-6.0 PS1
@@
 	1    0    0    -1
 $EndComp
+Wire Wire Line
+	5500 7500 5500 7550
+Wire Wire Line
+	5550 7400 5500 7400
+$Comp
+L EXTENSION:505567-0571 J8
+U 1 1 61909209
+P 2950 6050
+F 0 "J8" H 3350 6315 50  0000 C CNN
+F 1 "EXTIN" H 3350 6224 50  0000 C CNN
+F 2 "EXTENSION:5055670571" H 3600 6150 50  0001 L CNN
+F 3 "https://www.molex.com/pdm_docs/sd/5055670571_sd.pdf" H 3600 6050 50  0001 L CNN
+F 4 "Molex Micro-Lock PLUS 505567, 1.25mm Pitch, 5 Way, 1 Row, Right Angle PCB Header, Surface Mount" H 3600 5950 50  0001 L CNN "Description"
+F 5 "3" H 3600 5850 50  0001 L CNN "Height"
+F 6 "538-505567-0571" H 3600 5750 50  0001 L CNN "Mouser Part Number"
+F 7 "https://www.mouser.co.uk/ProductDetail/Molex/505567-0571?qs=gt1LBUVyoHnJxHrzoS78pw%3D%3D" H 3600 5650 50  0001 L CNN "Mouser Price/Stock"
+F 8 "Molex" H 3600 5550 50  0001 L CNN "Manufacturer_Name"
+F 9 "505567-0571" H 3600 5450 50  0001 L CNN "Manufacturer_Part_Number"
+	1    2950 6050
+	1    0    0    -1
+$EndComp
+Text GLabel 2900 6050 0    50   Input ~ 0
+PYRO1IN
+Text GLabel 2900 6150 0    50   Input ~ 0
+PYRO2IN
+Text GLabel 2900 6250 0    50   Input ~ 0
+BUZZ1IN
+Text GLabel 2900 6350 0    50   Input ~ 0
+BUZZ2IN
+Text GLabel 2900 6450 0    50   Input ~ 0
+GNDIN
+Wire Wire Line
+	2900 6450 2950 6450
+Wire Wire Line
+	2900 6350 2950 6350
+Wire Wire Line
+	2900 6250 2950 6250
+Wire Wire Line
+	2900 6150 2950 6150
+Wire Wire Line
+	2900 6050 2950 6050
 $EndSCHEMATC

Commit message: Worked again
Connections:
- net BUZZ1IN: now also IC1.9 (E_1), J1.4; no longer IC1.12 (E_2), J1.3
- net BUZZ2IN: now also IC1.12 (E_2), J1.3; no longer IC1.9 (E_1), J1.4
- net PYRO1IN: now also J1.2; no longer J1.1
- net PYRO2IN: now also J1.1; no longer J1.2
Changed lines of the file:
@@
 Text GLabel 8700 3300 0    50   Input ~ 0
 PYRO2IN
-Text GLabel 10050 3400 2    50   Input ~ 0
+Text GLabel 10050 3700 2    50   Input ~ 0
 BUZZ1IN
 Text GLabel 10050 3500 2    50   Input ~ 0
@@
 Text GLabel 10050 3600 2    50   Input ~ 0
 GNDIN
-Text GLabel 10050 3700 2    50   Input ~ 0
+Text GLabel 10050 3400 2    50   Input ~ 0
 BUZZ2IN
 Wire Wire Line
@@
 Wire Wire Line
 	9900 1300 9850 1300
+Text GLabel 1550 6150 0    50   Input ~ 0
+PYRO1IN
 Text GLabel 1550 6050 0    50   Input ~ 0
-PYRO1IN
-Text GLabel 1550 6150 0    50   Input ~ 0
 PYRO2IN
+Text GLabel 1550 6350 0    50   Input ~ 0
+BUZZ1IN
 Text GLabel 1550 6250 0    50   Input ~ 0
-BUZZ1IN
-Text GLabel 1550 6350 0    50   Input ~ 0
 BUZZ2IN
 Text GLabel 1550 6450 0    50   Input ~ 0

Commit message: Sent schematics to review
Parts:
- R2, R3: value 500 -> 510
Other:
- note added: "Ampli OP for pyro detection"
- note added: "Fuses for pyro channel"
- note added: "Input and Output connector"
- note added: "LEDs debug"
- note added: "MOSFETs for pyro + detection"
- note added: "Optocoupler"
- note added: "Voltage regulator for PWM"
- moved on the sheet: D1, D2, D3, D4, D5, IC1, J1, J2, J3, J4, J5, J6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

Commit message: t
Parts:
- added J9: 505567-0671, EXTENSION:5055670671, symbol EXTENSION:505567-0671
Connections:
- net BUZZ1IN: now also J9.3
- net BUZZ2IN: now also J9.4
- net GNDIN: now also J9.5
- net PYRO1IN: now also J9.1
- net PYRO2IN: now also J9.2
- new net 3V3IN: J9.6
Other:
- moved on the sheet: J8
Changed lines of the file:
@@
 L EXTENSION:505567-0571 J8
 U 1 1 61909209
-P 2550 5100
-F 0 "J8" H 2950 5365 50  0000 C CNN
-F 1 "EXTIN" H 2950 5274 50  0000 C CNN
-F 2 "EXTENSION:5055670571" H 3200 5200 50  0001 L CNN
-F 3 "https://www.molex.com/pdm_docs/sd/5055670571_sd.pdf" H 3200 5100 50  0001 L CNN
-F 4 "Molex Micro-Lock PLUS 505567, 1.25mm Pitch, 5 Way, 1 Row, Right Angle PCB Header, Surface Mount" H 3200 5000 50  0001 L CNN "Description"
-F 5 "3" H 3200 4900 50  0001 L CNN "Height"
-F 6 "538-505567-0571" H 3200 4800 50  0001 L CNN "Mouser Part Number"
-F 7 "https://www.mouser.co.uk/ProductDetail/Molex/505567-0571?qs=gt1LBUVyoHnJxHrzoS78pw%3D%3D" H 3200 4700 50  0001 L CNN "Mouser Price/Stock"
-F 8 "Molex" H 3200 4600 50  0001 L CNN "Manufacturer_Name"
-F 9 "505567-0571" H 3200 4500 50  0001 L CNN "Manufacturer_Part_Number"
-	1    2550 5100
+P -850 4900
+F 0 "J8" H -450 5165 50  0000 C CNN
+F 1 "EXTIN" H -450 5074 50  0000 C CNN
+F 2 "EXTENSION:5055670571" H -200 5000 50  0001 L CNN
+F 3 "https://www.molex.com/pdm_docs/sd/5055670571_sd.pdf" H -200 4900 50  0001 L CNN
+F 4 "Molex Micro-Lock PLUS 505567, 1.25mm Pitch, 5 Way, 1 Row, Right Angle PCB Header, Surface Mount" H -200 4800 50  0001 L CNN "Description"
+F 5 "3" H -200 4700 50  0001 L CNN "Height"
+F 6 "538-505567-0571" H -200 4600 50  0001 L CNN "Mouser Part Number"
+F 7 "https://www.mouser.co.uk/ProductDetail/Molex/505567-0571?qs=gt1LBUVyoHnJxHrzoS78pw%3D%3D" H -200 4500 50  0001 L CNN "Mouser Price/Stock"
+F 8 "Molex" H -200 4400 50  0001 L CNN "Manufacturer_Name"
+F 9 "505567-0571" H -200 4300 50  0001 L CNN "Manufacturer_Part_Number"
+	1    -850 4900
 	1    0    0    -1
 $EndComp
-Text GLabel 2500 5100 0    50   Input ~ 0
+Text GLabel -900 4900 0    50   Input ~ 0
 PYRO1IN
-Text GLabel 2500 5200 0    50   Input ~ 0
+Text GLabel -900 5000 0    50   Input ~ 0
 PYRO2IN
-Text GLabel 2500 5300 0    50   Input ~ 0
+Text GLabel -900 5100 0    50   Input ~ 0
 BUZZ1IN
-Text GLabel 2500 5400 0    50   Input ~ 0
+Text GLabel -900 5200 0    50   Input ~ 0
 BUZZ2IN
-Text GLabel 2500 5500 0    50   Input ~ 0
+Text GLabel -900 5300 0    50   Input ~ 0
 GNDIN
 Wire Wire Line
-	2500 5500 2550 5500
+	-900 5300 -850 5300
 Wire Wire Line
-	2500 5400 2550 5400
+	-900 5200 -850 5200
 Wire Wire Line
-	2500 5300 2550 5300
+	-900 5100 -850 5100
 Wire Wire Line
-	2500 5200 2550 5200
+	-900 5000 -850 5000
 Wire Wire Line
-	2500 5100 2550 5100
+	-900 4900 -850 4900
 Text Notes 4850 2250 0    50   ~ 0
 LEDs debug
@@
 Text Notes 9050 2250 0    50   ~ 0
 Ampli OP for pyro detection
+Text GLabel 2700 4750 0    50   Input ~ 0
+PYRO1IN
+Text GLabel 2700 4850 0    50   Input ~ 0
+PYRO2IN
+Text GLabel 2700 4950 0    50   Input ~ 0
+BUZZ1IN
+Text GLabel 2700 5050 0    50   Input ~ 0
+BUZZ2IN
+Text GLabel 2700 5150 0    50   Input ~ 0
+GNDIN
+Wire Wire Line
+	2700 5150 2750 5150
+Wire Wire Line
+	2700 5050 2750 5050
+Wire Wire Line
+	2700 4950 2750 4950
+Wire Wire Line
+	2700 4850 2750 4850
+Wire Wire Line
+	2700 4750 2750 4750
+$Comp
+L EXTENSION:505567-0671 J9
+U 1 1 61BAC7D6
+P 2750 4750
+F 0 "J9" H 3200 5015 50  0000 C CNN
+F 1 "505567-0671" H 3200 4924 50  0000 C CNN
+F 2 "EXTENSION:5055670671" H 3500 4850 50  0001 L CNN
+F 3 "https://componentsearchengine.com/Datasheets/1/505567-0671.pdf" H 3500 4750 50  0001 L CNN
+F 4 "Molex Micro-Lock PLUS 505567, 1.25mm Pitch, 6 Way, 1 Row, Right Angle PCB Header, Surface Mount" H 3500 4650 50  0001 L CNN "Description"
+F 5 "4.2" H 3500 4550 50  0001 L CNN "Height"
+F 6 "538-505567-0671" H 3500 4450 50  0001 L CNN "Mouser Part Number"
+F 7 "https://www.mouser.co.uk/ProductDetail/Molex/505567-0671?qs=gt1LBUVyoHmQuimOt9l14w%3D%3D" H 3500 4350 50  0001 L CNN "Mouser Price/Stock"
+F 8 "Molex" H 3500 4250 50  0001 L CNN "Manufacturer_Name"
+F 9 "505567-0671" H 3500 4150 50  0001 L CNN "Manufacturer_Part_Number"
+	1    2750 4750
+	1    0    0    -1
+$EndComp
+Text GLabel 2700 5250 0    50   Input ~ 0
+3V3IN
+Wire Wire Line
+	2700 5250 2750 5250
 $EndSCHEMATC

Commit message: a
Parts:
- removed J8: EXTIN, EXTENSION:5055670571, symbol EXTENSION:505567-0571
- J9: value 505567-0671 -> EXTIN
Connections:
- net 3V3IN: now also IC1.10 (C_5), IC1.11 (C_6)
- net BUZZ1IN: no longer IC1.9 (E_1), J9.3
- net BUZZ2IN: no longer IC1.12 (E_2), J9.4
- net GNDIN: no longer IC1.10 (C_5), IC1.11 (C_6)
- new net PDECT1IN: IC1.9 (E_1), J9.3
- new net PDECT2IN: IC1.12 (E_2), J9.4
Other:
- moved on the sheet: J1, J2, J3, J4, J5, J6, J7, J9

Commit message: aaa
Parts:
- removed J1: EXTIN, KRTEK_V2:2828345, symbol SamacSys_Parts:282834-5
Connections:
- net VINSERVO1 is gone; now on net VINSERVO2: J6.2, PS1.A5 (VOUT_1)
- net VCC: no longer PS1.D1 (PGOOD)
- no-connect marks 1 -> 2
Other:
- note added: "They have the same input as in datasheet\n"
Changed lines of the file:
@@
 Wire Wire Line
 	9900 1300 9850 1300
-Text GLabel 1200 5700 0    50   Input ~ 0
-PYRO1IN
-Text GLabel 1200 5600 0    50   Input ~ 0
-PYRO2IN
-Text GLabel 1200 5900 0    50   Input ~ 0
-BUZZ1IN
-Text GLabel 1200 5800 0    50   Input ~ 0
-BUZZ2IN
-Text GLabel 1200 6000 0    50   Input ~ 0
-GNDIN
-Wire Wire Line
-	1200 5600 1250 5600
-Wire Wire Line
-	1200 5700 1250 5700
-Wire Wire Line
-	1200 5800 1250 5800
-Wire Wire Line
-	1200 5900 1250 5900
-Wire Wire Line
-	1200 6000 1250 6000
 Text GLabel 1900 6700 3    50   Input ~ 0
 PYROTERMIN
@@
 Wire Wire Line
 	8800 5550 8750 5550
-Text GLabel 8500 4950 0    50   Input ~ 0
-VINSERVO1
 Text GLabel 8500 5450 0    50   Input ~ 0
 VINSERVO2
-Wire Wire Line
-	8500 4950 8800 4950
 Wire Wire Line
 	8500 5450 8800 5450
@@
 Wire Wire Line
 	10350 4650 10100 4650
-$Comp
-L power:VCC #PWR029
-U 1 1 618DFB2E
-P 10150 4750
-F 0 "#PWR029" H 10150 4600 50  0001 C CNN
-F 1 "VCC" H 10165 4923 50  0000 C CNN
-F 2 "" H 10150 4750 50  0001 C CNN
-F 3 "" H 10150 4750 50  0001 C CNN
-	1    10150 4750
-	0    1    1    0
-$EndComp
-Wire Wire Line
-	10100 4750 10150 4750
 $Comp
 L Device:R R18
@@
 	10650 5650 10700 5650
 Text GLabel 5200 6450 2    50   Input ~ 0
-VINSERVO1
+VINSERVO2
 $Comp
 L power:GND #PWR015
@@
 	1    5150 7050
 	-1   0    0    1
-$EndComp
-$Comp
-L SamacSys_Parts:282834-5 J1
-U 1 1 6181D2A8
-P 1250 5600
-F 0 "J1" H 1878 5446 50  0000 L CNN
-F 1 "EXTIN" H 1878 5355 50  0000 L CNN
-F 2 "KRTEK_V2:2828345" H 1900 5700 50  0001 L CNN
-F 3 "https://www.te.com/commerce/DocumentDelivery/DDEController?Action=showdoc&DocId=Customer+Drawing%7F282834%7FC1%7Fpdf%7FEnglish%7FENG_CD_282834_C1.pdf%7F282834-5" H 1900 5600 50  0001 L CNN
-F 4 "Conn Eurostyle Block HDR 5 POS 2.54mm Solder ST Thru-Hole 10A/Contact Carton" H 1900 5500 50  0001 L CNN "Description"
-F 5 "10.3" H 1900 5400 50  0001 L CNN "Height"
-F 6 "571-282834-5" H 1900 5300 50  0001 L CNN "Mouser Part Number"
-F 7 "https://www.mouser.co.uk/ProductDetail/TE-Connectivity/282834-5?qs=A%252Bip%252BNCYi6PY1Kyrkp4b4w%3D%3D" H 1900 5200 50  0001 L CNN "Mouser Price/Stock"
-F 8 "TE Connectivity" H 1900 5100 50  0001 L CNN "Manufacturer_Name"
-F 9 "282834-5" H 1900 5000 50  0001 L CNN "Manufacturer_Part_Number"
-	1    1250 5600
-	1    0    0    -1
 $EndComp
 Wire Wire Line
@@
 Text GLabel 7750 3800 2    50   Input ~ 0
 3V3IN
+NoConn ~ 10100 4750
+Text GLabel 8350 4950 0    50   Input ~ 0
+VINSERVO2
+Wire Wire Line
+	8350 4950 8800 4950
+Text Notes 5250 6300 0    50   ~ 0
+They have the same input as in datasheet\n
 $EndSCHEMATC

Commit message: duh
Connections:
- net PYRO1IN: now also J9.2; no longer J9.1
- net PYRO2IN: now also J9.1; no longer J9.2
Changed lines of the file:
@@
 Text Notes 9050 2250 0    50   ~ 0
 Ampli OP for pyro detection
+Text GLabel 2750 5350 0    50   Input ~ 0
+PYRO1IN
 Text GLabel 2750 5250 0    50   Input ~ 0
-PYRO1IN
-Text GLabel 2750 5350 0    50   Input ~ 0
 PYRO2IN
 Text GLabel 2750 5450 0    50   Input ~ 0
