File: POWER_BOARD/POWER_BOARD.sch (KiCad schematic (older format))
At the start: 37 parts, among them IC1 ILQ30, J2 ARM, J3 Pyro1, J4 Pyro2, J5 Servo2, J6 Servo1, J7 Batt, J9 EXTIN, Q1 IRL40B212, Q2 IRL40B212, U1 SF-1206HH10M-2, U2 SF-1206HH10M-2, U3 AS358AP

Commit message: Last changes
Parts:
- R10, R8: value 34k -> 93k
- R11: value 66k -> 7k
- R9: value 68k -> 7k
Changed lines of the file:
@@
 encoding utf-8
 Sheet 1 1
-Title ""
-Date ""
-Rev ""
-Comp ""
-Comment1 ""
+Title "The Power Board"
+Date "2022-01-02"
+Rev "R06"
+Comp "EPFL Rocket Team"
+Comment1 "EPFL Rocket Team all rights reserved"
 Comment2 ""
 Comment3 ""
@@
 P 2400 1300
 F 0 "R8" H 2330 1254 50  0000 R CNN
-F 1 "34k" H 2330 1345 50  0000 R CNN
+F 1 "93k" H 2330 1345 50  0000 R CNN
 F 2 "Resistor_SMD:R_0603_1608Metric" V 2330 1300 50  0001 C CNN
 F 3 "~" H 2400 1300 50  0001 C CNN
@@
 P 2400 1700
 F 0 "R9" H 2330 1654 50  0000 R CNN
-F 1 "68k" H 2330 1745 50  0000 R CNN
+F 1 "7k" H 2330 1745 50  0000 R CNN
 F 2 "Resistor_SMD:R_0603_1608Metric" V 2330 1700 50  0001 C CNN
 F 3 "~" H 2400 1700 50  0001 C CNN
@@
 P 2400 2900
 F 0 "R10" H 2330 2854 50  0000 R CNN
-F 1 "34k" H 2330 2945 50  0000 R CNN
+F 1 "93k" H 2330 2945 50  0000 R CNN
 F 2 "Resistor_SMD:R_0603_1608Metric" V 2330 2900 50  0001 C CNN
 F 3 "~" H 2400 2900 50  0001 C CNN
@@
 P 2400 3300
 F 0 "R11" H 2330 3254 50  0000 R CNN
-F 1 "66k" H 2330 3345 50  0000 R CNN
+F 1 "7k" H 2330 3345 50  0000 R CNN
 F 2 "Resistor_SMD:R_0603_1608Metric" V 2330 3300 50  0001 C CNN
 F 3 "~" H 2400 3300 50  0001 C CNN
